File: f1c100s/Power.sch (KiCad schematic (older format))
At the start: 19 parts, among them IC2 MCP1703T-2802E_CB, IC3 MCP1703T-2802E_CB, IC4 MCP1703T-2802E_CB, IC5 MCP1703T-2802E_CB, J1 USB_B_Micro

Commit message: All done i guess. DRC a little bit fuzzy but whatever.
Connections:
- net USB_DM renamed USB_N
- net USB_DP renamed USB_P
Changed lines of the file:
@@
 	8600 3550 9050 3550
 Text GLabel 8850 3750 2    50   Input ~ 0
-USB_DP
+USB_P
 Text GLabel 8850 3850 2    50   Input ~ 0
-USB_DM
+USB_N
 Wire Wire Line
 	9050 3550 9350 3550
